File: schema/mjGSM/mjGSM.sch (EAGLE design)
At the start: 20 parts, among them Q1 16MHz, SW1 SPST, U1 ATMEGA328P-PU, X2 PWR

Commit message: mod
Parts:
- removed SW1: SPST, gm-switches:SPST
- added RST: (no value), switch-omron:10-XX
- renumbered LED_STATUS to LED, SV1 to GSM, SV2 to FTDI, U1 to ATMEGA328P-PU, X2 to PWR
Connections:
- net GND: now also RST.P, RST.P1; no longer SW1.S
- net N$5: now also RST.S, RST.S1; no longer SW1.P

Commit message: mod
Parts:
- added C1, C2: 100nF, rcl:CPOL-EUE2-4
- added IC4: 7805T, linear:7805T
- GSM_PW: value GND -> (none)
- PWR: value PWR -> (none); SPICEPREFIX (none) -> X
Connections:
- removed net N$10: GSM.7, GSM_PW-1.KL
- removed net N$9: GSM.6, GSM_PW-2.KL
- new net 13V: C1.+, GSM_PW-1.KL, IC4.VI
- new net GSM5V: C2.+, GSM.7, IC4.VO
- new net GSMGND: C1.-, C2.-, GSM.6, GSM_PW-2.KL, IC4.GND
Other:
- note added: "Power"
- moved on the sheet: GSM_PW-1, GSM_PW-2
Changed lines of the file:
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@@
 <part name="GSM" library="con-lsta" library_urn="urn:adsk.eagle:library:161" deviceset="FE07-1" device="" package3d_urn="urn:adsk.eagle:package:8223/1" value="GSM"/>
 <part name="SUPPLY6" library="supply2" deviceset="GND" device=""/>
-<part name="GSM_PW" library="con-wago-500" library_urn="urn:adsk.eagle:library:195" deviceset="W237-102" device="" package3d_urn="urn:adsk.eagle:package:10688/1" value="GND"/>
-<part name="PWR" library="con-wago-500" library_urn="urn:adsk.eagle:library:195" deviceset="W237-102" device="" package3d_urn="urn:adsk.eagle:package:10688/1" value="PWR"/>
+<part name="GSM_PW" library="con-wago-500" library_urn="urn:adsk.eagle:library:195" deviceset="W237-102" device="" package3d_urn="urn:adsk.eagle:package:10688/1"/>
+<part name="PWR" library="con-wago-500" library_urn="urn:adsk.eagle:library:195" deviceset="W237-102" device="" package3d_urn="urn:adsk.eagle:package:10688/1">
+<attribute name="SPICEPREFIX" value="X"/>
+</part>
 <part name="I2C" library="con-wago-500" library_urn="urn:adsk.eagle:library:195" deviceset="W237-102" device="" package3d_urn="urn:adsk.eagle:package:10688/1"/>
 <part name="R1" library="my_rcl" deviceset="R-US_" device="0204/5" value="10K"/>
@@
 <part name="H4" library="holes" library_urn="urn:adsk.eagle:library:237" deviceset="MOUNT-HOLE" device="3.2" package3d_urn="urn:adsk.eagle:package:14275/1"/>
 <part name="RST" library="switch-omron" library_urn="urn:adsk.eagle:library:377" deviceset="10-XX" device="" package3d_urn="urn:adsk.eagle:package:27496/1"/>
+<part name="C1" library="rcl" deviceset="CPOL-EU" device="E2-4" value="100nF"/>
+<part name="C2" library="rcl" deviceset="CPOL-EU" device="E2-4" value="100nF"/>
+<part name="IC4" library="linear" deviceset="78*" device="T" technology="05"/>
 </parts>
 <sheets>
@@
 <text x="134.62" y="134.62" size="1.778" layer="91">VCC</text>
 <text x="142.24" y="147.32" size="1.778" layer="91">FTDI</text>
+<text x="175.26" y="93.98" size="3.81" layer="91">Power</text>
 </plain>
 <instances>
@@
 <instance part="GSM" gate="G$1" x="81.28" y="48.26" rot="MR0"/>
 <instance part="SUPPLY6" gate="GND" x="60.96" y="43.18" rot="R270"/>
-<instance part="GSM_PW" gate="-1" x="50.8" y="58.42"/>
-<instance part="GSM_PW" gate="-2" x="50.8" y="53.34"/>
+<instance part="GSM_PW" gate="-1" x="22.86" y="53.34"/>
+<instance part="GSM_PW" gate="-2" x="22.86" y="48.26"/>
 <instance part="PWR" gate="-1" x="17.78" y="71.12"/>
 <instance part="PWR" gate="-2" x="17.78" y="66.04"/>
@@
 <instance part="H4" gate="G$1" x="203.2" y="127"/>
 <instance part="RST" gate="1" x="104.14" y="104.14"/>
+<instance part="C1" gate="G$1" x="180.34" y="76.2"/>
+<instance part="C2" gate="G$1" x="205.74" y="76.2"/>
+<instance part="IC4" gate="A1" x="193.04" y="83.82"/>
 </instances>
 <busses>
@@
 </segment>
 </net>
-<net name="N$9" class="0">
-<segment>
-<pinref part="GSM_PW" gate="-2" pin="KL"/>
-<pinref part="GSM" gate="G$1" pin="6"/>
-<wire x1="55.88" y1="53.34" x2="73.66" y2="53.34" width="0.1524" layer="91"/>
-</segment>
-</net>
-<net name="N$10" class="0">
-<segment>
-<pinref part="GSM_PW" gate="-1" pin="KL"/>
-<pinref part="GSM" gate="G$1" pin="7"/>
-<wire x1="55.88" y1="58.42" x2="73.66" y2="55.88" width="0.1524" layer="91"/>
-</segment>
-</net>
 <net name="GSM_RX" class="0">
 <segment>
@@
 </segment>
 </net>
+<net name="GSM5V" class="0">
+<segment>
+<pinref part="IC4" gate="A1" pin="VO"/>
+<wire x1="203.2" y1="83.82" x2="205.74" y2="83.82" width="0.1524" layer="91"/>
+<pinref part="C2" gate="G$1" pin="+"/>
+<wire x1="205.74" y1="83.82" x2="223.52" y2="83.82" width="0.1524" layer="91"/>
+<wire x1="205.74" y1="78.74" x2="205.74" y2="83.82" width="0.1524" layer="91"/>
+<junction x="205.74" y="83.82"/>
+<label x="218.44" y="83.82" size="1.778" layer="95"/>
+</segment>
+<segment>
+<pinref part="GSM" gate="G$1" pin="7"/>
+<wire x1="73.66" y1="55.88" x2="63.5" y2="55.88" width="0.1524" layer="91"/>
+<label x="63.5" y="55.88" size="1.778" layer="95"/>
+</segment>
+</net>
+<net name="13V" class="0">
+<segment>
+<pinref part="IC4" gate="A1" pin="VI"/>
+<wire x1="182.88" y1="83.82" x2="180.34" y2="83.82" width="0.1524" layer="91"/>
+<pinref part="C1" gate="G$1" pin="+"/>
+<wire x1="180.34" y1="83.82" x2="170.18" y2="83.82" width="0.1524" layer="91"/>
+<wire x1="180.34" y1="78.74" x2="180.34" y2="83.82" width="0.1524" layer="91"/>
+<junction x="180.34" y="83.82"/>
+<label x="170.18" y="83.82" size="1.778" layer="95"/>
+</segment>
+<segment>
+<pinref part="GSM_PW" gate="-1" pin="KL"/>
+<wire x1="27.94" y1="53.34" x2="40.64" y2="53.34" width="0.1524" layer="91"/>
+<label x="30.48" y="53.34" size="1.778" layer="95"/>
+</segment>
+</net>
+<net name="GSMGND" class="0">
+<segment>
+<wire x1="170.18" y1="66.04" x2="180.34" y2="66.04" width="0.1524" layer="91"/>
+<pinref part="C1" gate="G$1" pin="-"/>
+<wire x1="180.34" y1="66.04" x2="193.04" y2="66.04" width="0.1524" layer="91"/>
+<wire x1="193.04" y1="66.04" x2="205.74" y2="66.04" width="0.1524" layer="91"/>
+<wire x1="205.74" y1="66.04" x2="220.98" y2="66.04" width="0.1524" layer="91"/>
+<wire x1="180.34" y1="71.12" x2="180.34" y2="66.04" width="0.1524" layer="91"/>
+<pinref part="IC4" gate="A1" pin="GND"/>
+<wire x1="193.04" y1="76.2" x2="193.04" y2="66.04" width="0.1524" layer="91"/>
+<pinref part="C2" gate="G$1" pin="-"/>
+<wire x1="205.74" y1="71.12" x2="205.74" y2="66.04" width="0.1524" layer="91"/>
+<junction x="180.34" y="66.04"/>
+<junction x="193.04" y="66.04"/>
+<junction x="205.74" y="66.04"/>
+<label x="170.18" y="66.04" size="1.778" layer="95"/>
+</segment>
+<segment>
+<pinref part="GSM" gate="G$1" pin="6"/>
+<wire x1="73.66" y1="53.34" x2="63.5" y2="53.34" width="0.1524" layer="91"/>
+<label x="63.5" y="53.34" size="1.778" layer="95"/>
+</segment>
+<segment>
+<pinref part="GSM_PW" gate="-2" pin="KL"/>
+<wire x1="27.94" y1="48.26" x2="40.64" y2="48.26" width="0.1524" layer="91"/>
+<label x="30.48" y="48.26" size="1.778" layer="95"/>
+</segment>
+</net>
